File: Tunnleing_Amp/Tunnleing_Amp.kicad_sch (KiCad schematic)
At the start: 11 parts, among them IC1 OPA928DT, J1 Conn_01x02_Pin

Commit message: Sent in V1.0 to JLC
Parts:
- removed C5: 4.7uF, 293D475X9035C2TE3:CAPPM6032X280N, symbol 293D475X9035C2TE3:293D475X9035C2TE3
- added C1: 4.7uF, 293D475X9035C2TE3:CAPPM6032X280N, symbol 293D475X9035C2TE3:293D475X9035C2TE3
Connections:
- net +15V: now also C3.1 (+), C6.1, IC1.5 (V+); no longer C4.1, IC1.4 (V-)
- net -15V: now also C4.1, IC1.4 (V-), C1.2 (-); no longer C3.1 (+), C6.1, IC1.5 (V+)
- net GND: now also C1.1 (+); no longer IC1.2 (GRD_1), IC1.7 (GRD_2)
- new net GRD: IC1.2 (GRD_1), IC1.7 (GRD_2)
