File: Mainboard/Mainboard.kicad_pcb (KiCad board)
At the start: 2 copper layers, 0 parts

Commit message: Mainboard grind
Parts:
- added C121: 330u 25V, Capacitor_THT:CP_Radial_D8.0mm_P3.50mm, F.Cu at (143.4, 102.1)
- added C122: 10u, Capacitor_SMD:C_1206_3216Metric, F.Cu at (152.8, 60.8)
- added C123: 10u, Capacitor_SMD:C_1206_3216Metric, F.Cu at (152.8, 64.2)
- added C124: 10u, Capacitor_SMD:C_1206_3216Metric, F.Cu at (152.8, 67.5)
- added C125: 10u, Capacitor_SMD:C_1206_3216Metric, F.Cu at (152.8, 70.9)
- added C126: 10u, Capacitor_SMD:C_1206_3216Metric, F.Cu at (152.8, 74.2)
- added C127: 10u, Capacitor_SMD:C_1206_3216Metric, F.Cu at (152.8, 77.6)
- added C128: 10u, Capacitor_SMD:C_1206_3216Metric, F.Cu at (158.4, 60.8)
- added C129: 10u, Capacitor_SMD:C_1206_3216Metric, F.Cu at (158.4, 64.2)
- added C130: 10u, Capacitor_SMD:C_1206_3216Metric, F.Cu at (158.4, 67.5)
- added C131: 10u, Capacitor_SMD:C_1206_3216Metric, F.Cu at (158.4, 70.9)
- added C132: 10u, Capacitor_SMD:C_1206_3216Metric, F.Cu at (158.4, 74.2)
- added C133: 10u, Capacitor_SMD:C_1206_3216Metric, F.Cu at (158.4, 77.6)
- added C134: 10u, Capacitor_SMD:C_1206_3216Metric, F.Cu at (164.1, 60.8)
- added C135: 10u, Capacitor_SMD:C_1206_3216Metric, F.Cu at (164.1, 64.2)
- added C136: 10u, Capacitor_SMD:C_1206_3216Metric, F.Cu at (164.1, 67.5)
- added C137: 10u, Capacitor_SMD:C_1206_3216Metric, F.Cu at (164.1, 70.9)
- added C77: 330u 25V, Capacitor_THT:CP_Radial_D8.0mm_P3.50mm, F.Cu at (143.4, 63.9)
- added C78: 330u 25V, Capacitor_THT:CP_Radial_D8.0mm_P3.50mm, F.Cu at (143.4, 73.5)
- added C81: 330u 25V, Capacitor_THT:CP_Radial_D8.0mm_P3.50mm, F.Cu at (143.4, 83.0)
- added C82: 330u 25V, Capacitor_THT:CP_Radial_D8.0mm_P3.50mm, F.Cu at (143.4, 92.6)
- added IC1: REF102AU_2K5, REF102AU_2K5:SOIC127P600X175-8N, F.Cu at (154.9, 118.7)
- added IC4: DAC8814IBDBT, DAC8814IBDBT:SOP65P780X200-28N, F.Cu at (145.4, 114.9)
- added J1: 5745782-6, 57457826:57457826, F.Cu at (126.7, 29.2)
- added J2: 5745782-6, 57457826:57457826, F.Cu at (126.7, 62.4)
- added J3: 5745782-6, 57457826:57457826, F.Cu at (126.7, 84.3)
- added JP12: Jumper, Jumper:SolderJumper-2_P1.3mm_Open_TrianglePad1.0x1.5mm, F.Cu at (116.7, 49.6)
- added JP29: Jumper, Jumper:SolderJumper-2_P1.3mm_Open_TrianglePad1.0x1.5mm, F.Cu at (116.7, 53.2)
- added JP30: Jumper, Jumper:SolderJumper-2_P1.3mm_Open_TrianglePad1.0x1.5mm, F.Cu at (150.8, 27.7)
- added JP31: Jumper, Jumper:SolderJumper-2_P1.3mm_Open_TrianglePad1.0x1.5mm, F.Cu at (150.8, 31.3)
- added JP32: Jumper, Jumper:SolderJumper-2_P1.3mm_Open_TrianglePad1.0x1.5mm, F.Cu at (150.8, 34.8)
- added JP33: Jumper, Jumper:SolderJumper-2_P1.3mm_Open_TrianglePad1.0x1.5mm, F.Cu at (150.8, 38.4)
- added TP1: TestPoint, TestPoint:TestPoint_Loop_D1.80mm_Drill1.0mm_Beaded, F.Cu at (98.3, 50.2)
- added TP2: TestPoint, TestPoint:TestPoint_Loop_D1.80mm_Drill1.0mm_Beaded, F.Cu at (98.3, 54.8)
- added TP3: TestPoint, TestPoint:TestPoint_Loop_D1.80mm_Drill1.0mm_Beaded, F.Cu at (102.9, 50.2)
- added TP4: TestPoint, TestPoint:TestPoint_Loop_D1.80mm_Drill1.0mm_Beaded, F.Cu at (102.9, 54.8)
- added TP5: TestPoint, TestPoint:TestPoint_Loop_D1.80mm_Drill1.0mm_Beaded, F.Cu at (107.6, 50.2)
- added TP6: TestPoint, TestPoint:TestPoint_Loop_D1.80mm_Drill1.0mm_Beaded, F.Cu at (107.6, 54.8)
- added TP7: TestPoint, TestPoint:TestPoint_Loop_D1.80mm_Drill1.0mm_Beaded, F.Cu at (112.2, 50.2)
- added TP8: TestPoint, TestPoint:TestPoint_Loop_D1.80mm_Drill1.0mm_Beaded, F.Cu at (112.2, 54.8)
- added U1: Teensy4.0, Teensy40:Teensy40, F.Cu at (115.6, 114.4)
- added U11: ADG419BR, Package_SO:SOIC-8_3.9x4.9mm_P1.27mm, F.Cu at (144.4, 29.3)
- added U12: ADG419BR, Package_SO:SOIC-8_3.9x4.9mm_P1.27mm, F.Cu at (144.4, 35.9)
- added U7: ADG419BR, Package_SO:SOIC-8_3.9x4.9mm_P1.27mm, F.Cu at (154.9, 112.2)
- added U8: LTC2326CMS-16-PBF, LTC2326-16:MSOP-16_MS_LIT, F.Cu at (143.9, 42.0)
- added U9: LT1469CS8-TRPBF, LT1469:SO-8_S_LIT, F.Cu at (152.9, 43.5)
