File: Mainboard/Mainboard.kicad_sch (KiCad schematic)
At the start: 13 parts, among them J4 5745782-6

Commit message: Mainboard grind
Parts:
- renumbered J4 to J1
Other:
- sheet ADC ports: added CNV_ADC, CS_ADC; removed CNV, ~CS_ADC
- sheet Connectors ports: added 1A_1, 1A_2, 1A_3, 1B_1, 1B_2, 1B_3, 2A_1, 2A_2, 2A_3, 2B_1, 2B_2, 2B_3, AIN+, AIN-, BIAS, IOUT+, IOUT-, T_Amp+, T_Amp-, Z+X, Z+Y, Z-X, Z-Y; removed none
- sheet StepperDrivers ports: added 1A_1, 1A_2, 1A_3, 1B_1, 1B_2, 1B_3, 2A_1, 2A_2, 2A_3, 2B_1, 2B_2, 2B_3; removed none
- sheet Teensy4.0 ports: added BUSY_ADC, CNV_ADC, CS_ADC, MISO_ADC, SCK_ADC; removed none
- moved on the sheet: C139, J1, JP12, JP29, R30
