File: Mainboard/DAC.kicad_sch (KiCad schematic)
At the start: 32 parts, among them IC1 REF102AU_2K5, IC4 DAC8814IBDBT, U2 TL072, U5 TL074, U6 TL074, U7 ADG419BR

Commit message: Mainboard grind
Other:
- moved on the sheet: IC4, R39

Commit message: working mainboard push!
Parts:
- removed C1: 10u, symbol Device:C_Small
- removed C9: 100u, symbol Device:C_Small
- added C40, C41, C42, C43, C44, C45, C46, C47: 100n, Capacitor_SMD:C_0805_2012Metric, symbol Device:C
- added C84: 10u, Capacitor_THT:CP_Radial_D5.0mm_P2.00mm, symbol Mainboard-rescue:CP_Small-Device
- added C85: 100u, Capacitor_THT:CP_Radial_D6.3mm_P2.50mm, symbol Mainboard-rescue:CP_Small-Device
- C16, C21, C22, C23: footprint (none) -> Capacitor_SMD:C_0805_2012Metric; Mouser Part Number (none) -> 80-C0805C332KCR
- C24, C25, C26, C27: footprint (none) -> Capacitor_SMD:C_0805_2012Metric; Mouser Part Number (none) -> 80-C0805C472J3GAUTO
- C8: footprint (none) -> Capacitor_SMD:C_0805_2012Metric; Mouser Part Number (none) -> 80-C0805C225K4R3123
- R19: footprint (none) -> Resistor_SMD:R_0805_2012Metric; Mouser Part Number (none) -> 755-ESR10EZPJ102
- R39: footprint (none) -> Resistor_SMD:R_0805_2012Metric; Mouser Part Number (none) -> 755-ESR10EZPD1002
- R40, R41, R42, R43: footprint (none) -> Resistor_SMD:R_0805_2012Metric; Mouser Part Number (none) -> 755-ESR10EZPF1501
- R50, R51, R52, R53, R54, R55, R56, R57, R58: footprint (none) -> Resistor_SMD:R_0805_2012Metric; Mouser Part Number (none) -> 667-ERA-6AED302V
- U2: footprint (none) -> Package_SO:SOIC-8-1EP_3.9x4.9mm_P1.27mm_EP2.29x3mm_ThermalVias; Mouser Part Number (none) -> 511-TL072BIDT
- U5, U6: footprint (none) -> Package_SO:SOIC-14_3.9x8.7mm_P1.27mm; Mouser Part Number (none) -> 511-TL074IYDT
- U7: Mouser Part Number (none) -> 584-ADG419BRZ-R
Connections:
- net +15V: now also C40.1, C42.1, C44.1, C46.1, C84.1
- net -15V: now also C41.2, C43.2, C45.2, C47.2
- net GND: now also C40.2, C41.1, C42.2, C43.1, C44.2, C45.1, C46.2, C47.1, C84.2, C85.2
- net at R19.2, U2.3 (+): now also C85.1
