File: Mainboard/Power.kicad_sch (KiCad schematic)
At the start: 21 parts

Commit message: working mainboard push!
Parts:
- removed C121: 330u 25V, Capacitor_THT:CP_Radial_D8.0mm_P3.50mm, symbol Mainboard-rescue:CP_Small-Device
- removed C126, C127, C128, C129, C133, C135, C136, C137: 10u, Capacitor_SMD:C_1206_3216Metric, symbol Device:C_Small
- C122, C123, C124, C125, C130, C131, C132, C134: value 10u -> 100n; footprint Capacitor_SMD:C_1206_3216Metric -> Capacitor_SMD:C_0805_2012Metric; Mouser Part Number (none) -> 80-C0805S104K1RACAUT
- C77, C78, C81, C82: value 330u 25V -> 10u; footprint Capacitor_THT:CP_Radial_D8.0mm_P3.50mm -> Capacitor_THT:CP_Radial_D5.0mm_P2.00mm; Mouser Part Number (none) -> 710-860020472003
Connections:
- net analog_-15V: no longer C130.1, C132.1, C134.1
- net analog_15V: no longer C131.2
- net analog_gnd: no longer C130.2, C131.1, C132.2, C134.2
- net digital_3V3: now also C130.1, C134.1
- net digital_5V: now also C131.2, C132.2
- net digital_gnd: now also C130.2, C131.1, C132.1, C134.2
Other:
- moved on the sheet: C122, C123, C124, C125
