File: Mainboard/StepperDrivers.kicad_sch (KiCad schematic)
At the start: 0 parts

Commit message: working mainboard push!
Parts:
- added A1, A2, A3: Pololu_Breakout_A4988, Module:Pololu_Breakout-16_15.2x20.3mm, symbol Driver_Motor:Pololu_Breakout_A4988
- added C28, C37, C38: 100n, Capacitor_SMD:C_0805_2012Metric, symbol Device:C_Small
- added C79, C80, C83: 100u, Capacitor_THT:CP_Radial_D6.3mm_P2.50mm, symbol Mainboard-rescue:CP_Small-Device
Connections:
- net 1A_1: now also A1.4 (1A)
- net 1A_2: now also A2.4 (1A)
- net 1A_3: now also A3.4 (1A)
- net 1B_1: now also A1.3 (1B)
- net 1B_2: now also A2.3 (1B)
- net 1B_3: now also A3.3 (1B)
- net 2A_1: now also A1.5 (2A)
- net 2A_2: now also A2.5 (2A)
- net 2A_3: now also A3.5 (2A)
- net 2B_1: now also A1.6 (2B)
- net 2B_2: now also A2.6 (2B)
- net 2B_3: now also A3.6 (2B)
- new net +3V3: A1.13 (~{RESET}), A1.14 (~{SLEEP}), A1.2 (VDD), A2.13 (~{RESET}), A2.14 (~{SLEEP}), A2.2 (VDD), A3.13 (~{RESET}), A3.14 (~{SLEEP}), A3.2 (VDD), C28.2, C37.2, C38.2
- new net +5V: A1.8 (VMOT), A2.8 (VMOT), A3.8 (VMOT), C79.1, C80.1, C83.1
- new net DIR_1: A1.16 (DIR)
- new net DIR_2: A2.16 (DIR)
- new net DIR_3: A3.16 (DIR)
- new net GND: A1.1 (GND), A1.7 (GND), A1.9 (~{ENABLE}), A2.1 (GND), A2.7 (GND), A2.9 (~{ENABLE}), A3.1 (GND), A3.7 (GND), A3.9 (~{ENABLE}), C28.1, C37.1, C38.1, C79.2, C80.2, C83.2
- new net STEP_1: A1.15 (STEP)
- new net STEP_2: A2.15 (STEP)
- new net STEP_3: A3.15 (STEP)
- no-connect marks 0 -> 9
Other:
- note added: "Decoupling"
- note added: "Stepper Drivers - Enable is pulled low to enable driver continuously - may pose thermal drift problems...."

Commit message: cad update
Other:
- moved on the sheet: C28, C37, C38, C79, C80, C83
