File: Power_Supply/regulation.kicad_sch (KiCad schematic)
At the start: 11 parts, among them IC1 TPS7A4700RGWR, IC2 TPS7A3301RGWR

Commit message: cad updates
Connections:
- net analog_-15v: now also IC2.1 (OUT_1); no longer IC2.3 (FB)
- net FB: now reaches C25.2, R30.1, R31.2
- net FB: now also IC2.3 (FB); no longer IC2.1 (OUT_1)
Other:
- moved on the sheet: C24, C25, R30, R31
Changed lines of the file:
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@@
 	(paper "A4")
+	(junction
+		(at 223.52 93.98)
+		(diameter 0)
+		(color 0 0 0 0)
+	)
 	(junction
 		(at 171.45 86.36)
@@
 	)
 	(junction
-		(at 223.52 83.82)
+		(at 231.14 86.36)
 		(diameter 0)
 		(color 0 0 0 0)
@@
 	)
 	(junction
-		(at 215.9 91.44)
-		(diameter 0)
-		(color 0 0 0 0)
-	)
-	(junction
-		(at 223.52 91.44)
+		(at 231.14 93.98)
 		(diameter 0)
 		(color 0 0 0 0)
@@
 	)
 	(junction
-		(at 215.9 83.82)
-		(diameter 0)
-		(color 0 0 0 0)
-	)
-	(junction
 		(at 96.52 87.63)
 		(diameter 0)
@@
 	)
 	(junction
-		(at 223.52 99.06)
+		(at 231.14 101.6)
 		(diameter 0)
 		(color 0 0 0 0)
@@
 	)
 	(junction
-		(at 231.14 83.82)
+		(at 238.76 86.36)
 		(diameter 0)
 		(color 0 0 0 0)
@@
 	(wire
 		(pts
-			(xy 219.71 99.06) (xy 223.52 99.06)
+			(xy 227.33 101.6) (xy 231.14 101.6)
 		)
 		(stroke
@@
 	(wire
 		(pts
-			(xy 231.14 83.82) (xy 231.14 87.63)
+			(xy 238.76 86.36) (xy 238.76 90.17)
 		)
 		(stroke
@@
 	(wire
 		(pts
-			(xy 223.52 96.52) (xy 223.52 99.06)
+			(xy 231.14 99.06) (xy 231.14 101.6)
 		)
 		(stroke
@@
 	(wire
 		(pts
-			(xy 215.9 83.82) (xy 223.52 83.82)
+			(xy 223.52 86.36) (xy 231.14 86.36)
 		)
 		(stroke
@@
 	(wire
 		(pts
+			(xy 222.25 93.98) (xy 223.52 93.98)
+		)
+		(stroke
+			(width 0)
+			(type default)
+		)
+	)
+	(wire
+		(pts
 			(xy 119.38 55.88) (xy 114.3 55.88)
 		)
@@
 	(wire
 		(pts
-			(xy 223.52 90.17) (xy 223.52 91.44)
+			(xy 231.14 92.71) (xy 231.14 93.98)
 		)
 		(stroke
@@
 	(wire
 		(pts
-			(xy 215.9 83.82) (xy 213.36 83.82)
-		)
-		(stroke
-			(width 0)
-			(type default)
-		)
-	)
-	(wire
-		(pts
 			(xy 203.2 109.22) (xy 203.2 111.76)
 		)
@@
 	(wire
 		(pts
-			(xy 223.52 83.82) (xy 223.52 85.09)
+			(xy 231.14 86.36) (xy 231.14 87.63)
 		)
 		(stroke
@@
 	(wire
 		(pts
-			(xy 215.9 91.44) (xy 223.52 91.44)
-		)
-		(stroke
-			(width 0)
-			(type default)
-		)
-	)
-	(wire
-		(pts
-			(xy 231.14 95.25) (xy 231.14 99.06)
-		)
-		(stroke
-			(width 0)
-			(type default)
-		)
-	)
-	(wire
-		(pts
-			(xy 213.36 86.36) (xy 210.82 86.36)
+			(xy 238.76 97.79) (xy 238.76 101.6)
 		)
 		(stroke
@@
 	(wire
 		(pts
-			(xy 223.52 83.82) (xy 231.14 83.82)
+			(xy 231.14 86.36) (xy 238.76 86.36)
 		)
 		(stroke
@@
 	(wire
 		(pts
-			(xy 210.82 91.44) (xy 215.9 91.44)
-		)
-		(stroke
-			(width 0)
-			(type default)
-		)
-	)
-	(wire
-		(pts
 			(xy 171.45 86.36) (xy 171.45 91.44)
 		)
@@
 	(wire
 		(pts
-			(xy 213.36 83.82) (xy 213.36 86.36)
-		)
-		(stroke
-			(width 0)
-			(type default)
-		)
-	)
-	(wire
-		(pts
 			(xy 99.06 87.63) (xy 96.52 87.63)
 		)
@@
 	(wire
 		(pts
+			(xy 223.52 93.98) (xy 231.14 93.98)
+		)
+		(stroke
+			(width 0)
+			(type default)
+		)
+	)
+	(wire
+		(pts
 			(xy 162.56 88.9) (xy 180.34 88.9)
 		)
@@
 	(wire
 		(pts
-			(xy 231.14 83.82) (xy 232.41 83.82)
+			(xy 238.76 86.36) (xy 240.03 86.36)
 		)
 		(stroke
@@
 	(wire
 		(pts
-			(xy 223.52 99.06) (xy 231.14 99.06)
+			(xy 231.14 101.6) (xy 238.76 101.6)
 		)
 		(stroke
@@
 			(width 0)
 			(type default)
+		)
+	)
+	(label "FB"
+		(at 210.82 86.36 0)
+		(effects
+			(font
+				(size 1.27 1.27)
+			)
+			(justify left bottom)
+		)
+	)
+	(label "FB"
+		(at 222.25 93.98 180)
+		(effects
+			(font
+				(size 1.27 1.27)
+			)
+			(justify right bottom)
+		)
+	)
+	(label "OUT_1"
+		(at 210.82 91.44 0)
+		(effects
+			(font
+				(size 1.27 1.27)
+			)
+			(justify left bottom)
+		)
+	)
+	(label "OUT_1"
+		(at 223.52 86.36 180)
+		(effects
+			(font
+				(size 1.27 1.27)
+			)
+			(justify right bottom)
 		)
 	)
@@
 	(hierarchical_label "gnd"
 		(shape input)
-		(at 219.71 99.06 180)
+		(at 227.33 101.6 180)
 		(effects
 			(font
@@
 	(hierarchical_label "analog_-15v"
 		(shape input)
-		(at 232.41 83.82 0)
+		(at 240.03 86.36 0)
 		(effects
 			(font
@@
 	(symbol
 		(lib_id "Device:C")
-		(at 215.9 87.63 0)
+		(at 223.52 90.17 0)
 		(unit 1)
 		(exclude_from_sim no)
@@
 		(dnp no)
 		(property "Reference" "C25"
-			(at 222.504 86.106 0)
+			(at 230.124 88.646 0)
 			(effects
 				(font
@@
 		)
 		(property "Value" "10n"
-			(at 223.012 88.392 0)
+			(at 230.632 90.932 0)
 			(effects
 				(font
@@
 		)
 		(property "Footprint" "Capacitor_SMD:C_0603_1608Metric"
-			(at 216.8652 91.44 0)
+			(at 224.4852 93.98 0)
 			(effects
 				(font
@@
 		)
 		(property "Datasheet" "https://www.reichelt.de/vielschicht-kerko-4-7-f-16v-125-c-kem-x7r0805-4-7u-p207081.html?&trstct=pol_3"
-			(at 215.9 87.63 0)
+			(at 223.52 90.17 0)
 			(effects
 				(font
@@
 		)
 		(property "Description" ""
-			(at 215.9 87.63 0)
+			(at 223.52 90.17 0)
 			(effects
 				(font
@@
 		)
 		(property "Mouser Part Number" "581-06033C103KAZ2A"
-			(at 215.9 87.63 0)
+			(at 223.52 90.17 0)
 			(effects
 				(font
@@
 	(symbol
 		(lib_id "Device:R_Small")
-		(at 223.52 93.98 180)
+		(at 231.14 96.52 180)
 		(unit 1)
 		(exclude_from_sim no)
@@
 		(dnp no)
 		(property "Reference" "R31"
-			(at 219.964 92.71 0)
+			(at 227.584 95.25 0)
 			(effects
 				(font
@@
 		)
 		(property "Value" "105k"
-			(at 221.234 94.742 0)
+			(at 228.854 97.282 0)
 			(effects
 				(font
@@
 		)
 		(property "Footprint" "Resistor_SMD:R_0805_2012Metric"
-			(at 223.52 93.98 0)
+			(at 231.14 96.52 0)
 			(effects
 				(font
@@
 		)
 		(property "Datasheet" "~"
-			(at 223.52 93.98 0)
+			(at 231.14 96.52 0)
 			(effects
 				(font
@@
 		)
 		(property "Description" ""
-			(at 223.52 93.98 0)
+			(at 231.14 96.52 0)
 			(effects
 				(font
@@
 		)
 		(property "Mouser Part Number" "279-RQ73C2A105KBTD"
-			(at 223.52 93.98 0)
+			(at 231.14 96.52 0)
 			(effects
 				(font
@@
 	(symbol
 		(lib_id "Supply-Board-rescue:CP-Device")
-		(at 231.14 91.44 180)
+		(at 238.76 93.98 180)
 		(unit 1)
 		(exclude_from_sim no)
@@
 		(dnp no)
 		(property "Reference" "C24"
-			(at 235.458 89.408 0)
+			(at 243.078 91.948 0)
 			(effects
 				(font
@@
 		)
 		(property "Value" "47u"
-			(at 234.95 91.694 0)
+			(at 242.57 94.234 0)
 			(effects
 				(font
@@
 		)
 		(property "Footprint" "Capacitor_Tantalum_SMD:CP_EIA-7343-31_Kemet-D"
-			(at 231.14 91.44 0)
+			(at 238.76 93.98 0)
 			(effects
 				(font
@@
 		)
 		(property "Datasheet" "https://www.reichelt.de/smd-tantal-10-f-16v-125-c-t491c-10u-16-p206468.html?&trstct=pol_3"
-			(at 231.14 91.44 0)
+			(at 238.76 93.98 0)
 			(effects
 				(font
@@
 		)
 		(property "Description" ""
-			(at 231.14 91.44 0)
+			(at 238.76 93.98 0)
 			(effects
 				(font
@@
 		)
 		(property "Mouser Part Number" "80-T491D476K020"
-			(at 228.854 80.01 0)
+			(at 236.474 82.55 0)
 			(effects
 				(font
@@
 	(symbol
 		(lib_id "Device:R_Small")
-		(at 223.52 87.63 180)
+		(at 231.14 90.17 180)
 		(unit 1)
 		(exclude_from_sim no)
@@
 		(dnp no)
 		(property "Reference" "R30"
-			(at 229.616 86.106 0)
+			(at 237.236 88.646 0)
 			(effects
 				(font
@@
 		)
 		(property "Value" "1.24M"
-			(at 231.14 88.138 0)
+			(at 238.76 90.678 0)
 			(effects
 				(font
@@
 		)
 		(property "Footprint" "Resistor_SMD:R_0805_2012Metric"
-			(at 223.52 87.63 0)
+			(at 231.14 90.17 0)
 			(effects
 				(font
@@
 		)
 		(property "Datasheet" "~"
-			(at 223.52 87.63 0)
+			(at 231.14 90.17 0)
 			(effects
 				(font
@@
 		)
 		(property "Description" ""
-			(at 223.52 87.63 0)
+			(at 231.14 90.17 0)
 			(effects
 				(font
@@
 		)
 		(property "Mouser Part Number" "71-CRCW08051M24FKEA"
-			(at 223.52 87.63 0)
-			(effects
-				(font
+			(at 231.14 90.17 0)
+			(effects
+				(font
