File: Power_Supply/Power_Supply.kicad_pcb (KiCad board)
At the start: 4 copper layers, 165.7 x 132 mm, 82 parts, among them IC1 TPS7A4700RGWR, IC2 TPS7A3301RGWR, J1 Conn_01x03_Pin, J2 Conn_01x03_Pin, J3 Conn_01x03_Pin, J4 5745782-6, J7 1287, J8 1287, J9 1287, K2 G5LE-1, Q1 2N7000, U3 Fuse, 1A, U4 Fuse, 5A, U5 traco_TSR_0.5-2433, U6 LM75C

Commit message: Analog Circuit V1.0
Connections:
- net /SCL renamed /PS_Temp_SCL
- net /SDA renamed /PS_Temp_SDA
- net /analog/piezo_gnd renamed /analog_gnd

Commit message: cad updates
Connections:
- C25 pad 2: Net-(IC2-OUT_1) -> /regulation/FB
- IC2 pad 1: Net-(IC2-OUT_1) -> /analog_-15V
- IC2 pad 3: /analog_-15V -> /regulation/FB
- R30 pad 1: Net-(IC2-OUT_1) -> /regulation/FB
- R31 pad 2: Net-(IC2-OUT_1) -> /regulation/FB
Routing:
- net Net-(IC2-OUT_1): track 15.3 -> 0.00 mm
- net /regulation/FB: track 0.00 -> 13.0 mm
- net /analog_-15V: track 18.2 -> 19.2 mm
Changed lines of the file:
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@@
 	(net 11 "Net-(D10-K)")
 	(net 12 "/digital_3V3")
-	(net 13 "Net-(IC2-OUT_1)")
+	(net 13 "/regulation/FB")
 	(net 14 "/analog_15V")
 	(net 15 "Net-(IC2-NR{slash}SS)")
@@
 			(layers "F.Cu" "F.Mask" "F.Paste")
 			(roundrect_rratio 0.25)
-			(net 13 "Net-(IC2-OUT_1)")
+			(net 13 "/regulation/FB")
 			(pintype "passive")
 		)
@@
 			(size 0.35 1.05)
 			(layers "F.Cu" "F.Mask" "F.Paste")
-			(net 13 "Net-(IC2-OUT_1)")
+			(net 16 "/analog_-15V")
 			(pinfunction "OUT_1")
 			(pintype "passive")
@@
 			(size 0.35 1.05)
 			(layers "F.Cu" "F.Mask" "F.Paste")
-			(net 16 "/analog_-15V")
+			(net 13 "/regulation/FB")
 			(pinfunction "FB")
 			(pintype "passive")
@@
 			(layers "F.Cu" "F.Mask" "F.Paste")
 			(roundrect_rratio 0.243902)
-			(net 13 "Net-(IC2-OUT_1)")
+			(net 13 "/regulation/FB")
 			(pintype "passive")
 		)
@@
 			(layers "F.Cu" "F.Mask" "F.Paste")
 			(roundrect_rratio 0.243902)
-			(net 13 "Net-(IC2-OUT_1)")
+			(net 13 "/regulation/FB")
 			(pintype "passive")
 		)
@@
 	)
 	(segment
-		(start 142.19 35.19)
-		(end 141.29 34.29)
-		(width 0.3)
-		(layer "F.Cu")
-		(net 13)
-	)
-	(segment
 		(start 139.115 42.54)
 		(end 141.215 42.54)
@@
 	)
 	(segment
-		(start 141.29 34.29)
-		(end 140.24 34.29)
-		(width 0.3)
-		(layer "F.Cu")
-		(net 13)
-	)
-	(segment
 		(start 138.74 51.94)
 		(end 139.79 51.94)
@@
 		(width 0.3)
 		(layer "F.Cu")
+		(net 16)
+	)
+	(segment
+		(start 141.29 34.29)
+		(end 140.24 34.29)
+		(width 0.3)
+		(layer "F.Cu")

Commit message: final
Routing:
- net /regulation/FB: track 13.0 -> 14.4 mm, vias 0 -> 1
- net /analog_-15V: track 19.2 -> 17.9 mm, vias 17 -> 16
Changed lines of the file:
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@@
 			(psa4output no)
 			(plot_black_and_white yes)
-			(plotinvisibletext no)
 			(sketchpadsonfab no)
 			(plotpadnumbers no)
@@
 	)
 	(segment
+		(start 141.59 32.99)
+		(end 140.24 32.99)
+		(width 0.3)
+		(layer "F.Cu")
+		(net 13)
+	)
+	(segment
 		(start 142.19 37.49)
 		(end 142.19 39.9275)
@@
 		(net 13)
 	)
+	(via
+		(at 141.59 32.99)
+		(size 0.6)
+		(drill 0.3)
+		(layers "F.Cu" "B.Cu")
+		(net 13)
+	)
 	(segment
 		(start 138.74 51.94)
@@
 	)
 	(segment
-		(start 141.59 32.99)
-		(end 140.24 32.99)
-		(width 0.3)
-		(layer "F.Cu")
-		(net 16)
-	)
-	(segment
 		(start 141.29 34.29)
 		(end 140.24 34.29)
@@
 		(size 0.6)
 		(drill 0.3)
-		(layers "F.Cu" "B.Cu")
-		(net 16)
-	)
-	(via
-		(at 141.59 32.99)
-		(size 0.6)
-		(drill 0.3)
