File: Power_Supply/Power_Supply.kicad_sch (KiCad schematic)
At the start: 69 parts, among them J1 Conn_01x03_Pin, J2 Conn_01x03_Pin, J3 Conn_01x03_Pin, J4 5745782-6, J7 1287, J8 1287, J9 1287, K2 G5LE-1, Q1 2N7000, U3 Fuse, 1A, U4 Fuse, 5A, U5 traco_TSR_0.5-2433, U6 LM75C

Commit message: final
Other:
- moved on the sheet: R20
Changed lines of the file:
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@@
 	(wire
 		(pts
-			(xy 102.87 135.89) (xy 102.87 142.24)
+			(xy 102.87 138.43) (xy 102.87 142.24)
 		)
 		(stroke
@@
 	(wire
 		(pts
-			(xy 102.87 128.27) (xy 102.87 130.81)
+			(xy 102.87 128.27) (xy 102.87 133.35)
 		)
 		(stroke
@@
 	(symbol
 		(lib_id "Device:R_Small")
-		(at 102.87 133.35 180)
+		(at 102.87 135.89 180)
 		(unit 1)
 		(exclude_from_sim no)
@@
 		(dnp no)
 		(property "Reference" "R20"
-			(at 101.346 131.572 0)
+			(at 101.346 132.588 0)
 			(effects
 				(font
@@
 		)
 		(property "Value" "56k"
-			(at 101.346 134.366 0)
+			(at 101.346 135.128 0)
 			(effects
 				(font
@@
 		)
 		(property "Footprint" "Resistor_SMD:R_0805_2012Metric"
-			(at 102.87 133.35 0)
+			(at 102.87 135.89 0)
 			(effects
 				(font
@@
 		)
 		(property "Datasheet" "~"
-			(at 102.87 133.35 0)
+			(at 102.87 135.89 0)
 			(effects
 				(font
@@
 		)
 		(property "Description" ""
-			(at 102.87 133.35 0)
+			(at 102.87 135.89 0)
 			(effects
 				(font
@@
 		)
 		(property "Mouser Part Number" "755-ESR10EZPF5602"
-			(at 102.87 133.35 0)
+			(at 102.87 135.89 0)
 			(effects
 				(font
